File: catlink-tracker-pcb/catlink-tracker-pcb.kicad_pcb (KiCad board)
At the start: 4 copper layers, 17.6 x 35.1 mm, 34 parts, among them J1 S2B-PH-K, J2 U.FL, U1 STM32L412K8Tx, U2 TLV75530PDBV, U3 Ai-Thinker-Ra-01S, U4 E108-GN03

Commit message: Changed logo, added pin 1 silkscreen for ESD diode
Parts:
- moved G*** 0.72 mm to (120.0, 103.9)
