File: catlink-gateway-pcb-eval/catlink-gateway-pcb-eval.kicad_pcb (KiCad board)
At the start: 4 copper layers, 70 x 97.5 mm, 52 parts, among them J1 TYPE-C-31-M-12, J2 Conn_02x05_Odd_Even, J3 Conn_02x05_Odd_Even, SW1 SW_SPDT, U1 ESP32-C3-MINI-1, U2 TPD4E05U06DQA, U3 TP4056-42-ESOP8, U4 TPS2116DRL, U5 TLV75901PDRV, U6 Ai-Thinker-Ra-01S

Commit message: Added state LED and IO9 switch
Parts:
- added D8: RED, LED_SMD:LED_0805_2012Metric, F.Cu at (181.2, 89.8)
- added R21: 1k2, Resistor_SMD:R_0603_1608Metric, F.Cu at (179.4, 92.2)
- added R22: 10k, Resistor_SMD:R_0603_1608Metric, F.Cu at (177.2, 124.2)
- added R23: 10k, Resistor_SMD:R_0603_1608Metric, F.Cu at (177.2, 129.8)
- added SW2: SW_SPDT, Button_Switch_THT:SW_Slide_SPDT_Angled_CK_OS102011MA1Q, F.Cu at (181.7, 129.0)
- R11, R20: value 200 -> 1k2; footprint Resistor_SMD:R_0805_2012Metric -> Resistor_SMD:R_0603_1608Metric
- R12: value 300 -> 1k2; footprint Resistor_SMD:R_0805_2012Metric -> Resistor_SMD:R_0603_1608Metric
- moved R3 1.20 mm to (167.2, 70.8)
Connections:
- U1 pad 18: /DIO3 -> Net-(U1-IO4)
- U1 pad 23: unconnected-(U1-IO9-Pad23) -> /IO9
Routing:
- net /IO9: track 0.00 -> 85.2 mm, vias 0 -> 3
- net Net-(U1-IO4): track 0.00 -> 32.2 mm, vias 0 -> 4
- net /DIO3: track 32.2 -> 7.04 mm, vias 2 -> 0
- net +3V0: track 4.71 -> 11.2 mm, vias 11 -> 12
- net GND: track 9.48 -> 14.1 mm
- net Net-(SW2-C): track 0.00 -> 4.46 mm
- net Net-(SW2-A): track 0.00 -> 4.46 mm
- net Net-(D8-K): track 0.00 -> 2.45 mm
Other:
- board text added: "SPI BOOT ↑"
- board text added: "USB-JTAG BOOT ↓"
