File: catlink-gateway-pcb-eval/catlink-gateway-pcb-eval.kicad_sch (KiCad schematic)
At the start: 51 parts, among them J1 TYPE-C-31-M-12, J2 Conn_02x05_Odd_Even, J3 Conn_02x05_Odd_Even, SW1 SW_SPDT, U1 ESP32-C3-MINI-1, U2 TPD4E05U06DQA, U3 TP4056-42-ESOP8, U4 TPS2116DRL, U5 TLV75901PDRV, U6 Ai-Thinker-Ra-01S

Commit message: Added state LED and IO9 switch
Parts:
- added D8: RED, LED_SMD:LED_0805_2012Metric, symbol Device:LED
- added R21: 1k2, Resistor_SMD:R_0603_1608Metric, symbol Device:R
- added R22, R23: 10k, Resistor_SMD:R_0603_1608Metric, symbol Device:R
- added SW2: SW_SPDT, Button_Switch_THT:SW_Slide_SPDT_Angled_CK_OS102011MA1Q, symbol Switch:SW_SPDT
- R11, R20: value 200 -> 1k2; footprint Resistor_SMD:R_0805_2012Metric -> Resistor_SMD:R_0603_1608Metric
- R12: value 300 -> 1k2; footprint Resistor_SMD:R_0805_2012Metric -> Resistor_SMD:R_0603_1608Metric
Connections:
- net +3V0: now also D8.2 (A), R22.1
- net DIO3: no longer U1.18 (IO4)
- net GND: now also R23.2
- net IO9: now reaches U1.23 (IO9)
- net IO9: now also SW2.2 (B)
- new net: R21.2, U1.18 (IO4)
- new net: D8.1 (K), R21.1
- new net: R22.2, SW2.3 (C)
- new net: R23.1, SW2.1 (A)
- no-connect marks 6 -> 5
